File: M6/CPR Machine Schematic/Power.kicad_sch (KiCad schematic)
At the start: 51 parts, among them J1 Battery 22.2V IN, J2 5V Spare Headers, J3 Power Switch, J4 3V3 Spare Headers, J5 12 Spare headers, J6 Battery Spare headers, J7 GND Spare Headers, Q1 2N3904, Q2 AO3407A, Q4 DMMT5401 PNP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

Commit message: Final PCB
Parts:
- added H1, H2, H3, H4: MountingHole, MountingHole:MountingHole_2.7mm_M2.5_Pad, symbol Mechanical:MountingHole
- F1: value 5A -> 4A; digikey 5923-C1F5CT-ND -> 5923-0685T4000-01CT-ND
- Q2: value AO3407A -> SSM3J332R; MANUFACTURER Diodes Inc. -> (none); MAXIMUM_PACKAGE_HEIGHT 1.1mm -> (none); PARTREV 09/2018 -> (none); STANDARD IPC-7351B -> (none); digikey 785-1006-1-ND -> SSM3J332RLFCT-ND

Commit message: Start of Board V2
Parts:
- added Contactor1: G5Q-1A, Relay_THT:Relay_SPST_Omron-G5Q-1A, symbol Relay:G5Q-1A
- added Flyback1: 1N4001, Diode_THT:D_DO-41_SOD81_P10.16mm_Horizontal, symbol Diode:1N4001
- added J14: Battery, symbol Connector:Conn_01x02_Socket
- added SW1: SW_SPST, symbol Switch:SW_SPST
Connections:
- net +12V: now also Contactor1.1, Flyback1.1 (K)
- net Battery +: now also Contactor1.2
- net From Switch: now also SW1.2 (B)
- net GND: now also Contactor1.5, Flyback1.2 (A), J14.2 (Pin_2)
- new net: Contactor1.3, J14.1 (Pin_1), SW1.1 (A)
Other:
- note added: "Power Cable - NOT ON BOARD"
- moved on the sheet: J3, U4

Commit message: Fixed edge cuts
Parts:
- removed H2: MountingHole, MountingHole:MountingHole_2.7mm_M2.5_Pad, symbol Mechanical:MountingHole
Other:
- moved on the sheet: H3, H4
Changed lines of the file:
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@@
 	)
 	(symbol
-		(lib_id "Mechanical:MountingHole")
-		(at 266.7 21.59 0)
-		(unit 1)
-		(exclude_from_sim no)
-		(in_bom no)
-		(on_board yes)
-		(dnp no)
-		(fields_autoplaced yes)
-		(property "Reference" "H2"
-			(at 269.24 20.3199 0)
-			(effects
-				(font
-					(size 1.27 1.27)
-				)
-				(justify left)
-			)
-		)
-		(property "Value" "MountingHole"
-			(at 269.24 22.8599 0)
-			(effects
-				(font
-					(size 1.27 1.27)
-				)
-				(justify left)
-			)
-		)
-		(property "Footprint" "MountingHole:MountingHole_2.7mm_M2.5_Pad"
-			(at 266.7 21.59 0)
-			(effects
-				(font
-					(size 1.27 1.27)
-				)
-				(hide yes)
-			)
-		)
-		(property "Datasheet" "~"
-			(at 266.7 21.59 0)
-			(effects
-				(font
-					(size 1.27 1.27)
-				)
-				(hide yes)
-			)
-		)
-		(property "Description" "Mounting Hole without connection"
-			(at 266.7 21.59 0)
-			(effects
-				(font
-					(size 1.27 1.27)
-				)
-				(hide yes)
-			)
-		)
-		(instances
-			(project "CPR Machine Schematic"
-				(path "/8991fc77-975f-4978-a089-6b2a5e33f59b/390cafbd-c317-4387-95c3-e11405a1139f"
-					(reference "H2")
-					(unit 1)
-				)
-			)
-		)
-	)
-	(symbol
 		(lib_id "power:+5V")
 		(at 45.72 163.83 0)
@@
 	(symbol
 		(lib_id "Mechanical:MountingHole")
-		(at 266.7 31.75 0)
+		(at 266.7 26.67 0)
 		(unit 1)
 		(exclude_from_sim no)
@@
 		(fields_autoplaced yes)
 		(property "Reference" "H4"
-			(at 269.24 30.4799 0)
+			(at 269.24 25.3999 0)
 			(effects
 				(font
@@
 		)
 		(property "Value" "MountingHole"
-			(at 269.24 33.0199 0)
+			(at 269.24 27.9399 0)
 			(effects
 				(font
@@
 		)
 		(property "Footprint" "MountingHole:MountingHole_2.7mm_M2.5_Pad"
-			(at 266.7 31.75 0)
+			(at 266.7 26.67 0)
 			(effects
 				(font
@@
 		)
 		(property "Datasheet" "~"
-			(at 266.7 31.75 0)
+			(at 266.7 26.67 0)
 			(effects
 				(font
@@
 		)
 		(property "Description" "Mounting Hole without connection"
-			(at 266.7 31.75 0)
+			(at 266.7 26.67 0)
 			(effects
 				(font
@@
 	(symbol
 		(lib_id "Mechanical:MountingHole")
-		(at 266.7 26.67 0)
+		(at 266.7 21.59 0)
 		(unit 1)
 		(exclude_from_sim no)
@@
 		(fields_autoplaced yes)
 		(property "Reference" "H3"
-			(at 269.24 25.3999 0)
+			(at 269.24 20.3199 0)
 			(effects
 				(font
@@
 		)
 		(property "Value" "MountingHole"
-			(at 269.24 27.9399 0)
+			(at 269.24 22.8599 0)
 			(effects
 				(font
@@
 		)
 		(property "Footprint" "MountingHole:MountingHole_2.7mm_M2.5_Pad"
-			(at 266.7 26.67 0)
+			(at 266.7 21.59 0)
 			(effects
 				(font
@@
 		)
 		(property "Datasheet" "~"
-			(at 266.7 26.67 0)
+			(at 266.7 21.59 0)
 			(effects
 				(font
@@
 		)
 		(property "Description" "Mounting Hole without connection"
-			(at 266.7 26.67 0)
+			(at 266.7 21.59 0)
 			(effects
 				(font

Commit message: Board V2
Parts:
- added COUT2: 23.7 uF, Capacitor_SMD:C_1210_3225Metric_Pad1.33x2.70mm_HandSolder, symbol Device:C
- added F3: 40A, Fuse:Fuse_1206_3216Metric_Pad1.42x1.75mm_HandSolder, symbol Device:Fuse
- added J16: Motor Driver, symbol Connector:Conn_01x02_Socket
- added Q5: DMMT5401 PNP, 2679:SOT95P285X140-6N, symbol 2679:DMMT5401 PNP
- added Q8: DMG2305UX-EV, Package_TO_SOT_SMD:SOT-23_Handsoldering, symbol 2679:DMG2305UX-13 MOSFET
- added R25: 10 kOhm, Resistor_SMD:R_1206_3216Metric_Pad1.30x1.75mm_HandSolder, symbol Device:R_US
- added R26: 47 kOhm, Resistor_SMD:R_1206_3216Metric_Pad1.30x1.75mm_HandSolder, symbol Device:R_US
- COUT1: value 47 uF -> 23.7 uF; footprint Capacitor_THT:CP_Radial_D8.0mm_P3.50mm -> Capacitor_SMD:C_1210_3225Metric_Pad1.33x2.70mm_HandSolder; digikey 732-6324-1-ND -> 490-5312-1-ND
- Contactor1, Flyback1, J14, SW1: now left out of the parts list
Connections:
- net +12V: now also Contactor1.2, F3.1
- net +5V: now also Q5.5, Q8.2; no longer C3.2, COUT1.1, L1.1, R1.1
- net Battery +: now also F3.2, J16.1 (Pin_1); no longer Contactor1.2
- net GND: now also COUT2.2, J16.2 (Pin_2), R25.2, R26.2
- new net: Q5.4, Q8.1, R26.1
- new net: Q5.1, Q5.2, Q5.3, R25.1
- new net Reg OUT: C3.2, COUT1.1, COUT2.1, L1.1, Q5.6, Q8.3, R1.1
Other:
- note added: "Regulator 0V Diode"
- note added: "To prevent backdriving when Raspi is plugged in"
- moved on the sheet: C1, C10, C11, C12, C3, C5, C7, C8, C9, CIN1, CIN2, COUT1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

Commit message: Board V2 Final
Parts:
- C3, F1, J1, J3, L1, Q4, Q5, R1, R10, R14, R2, R26, R3, R9, U4: now left out of the parts list
- C8, CIN1, CIN2: Notes (none) -> Have: 4
- LED1, LED2, LED3, LED4: Notes (none) -> Have: 2
- U2, U6: Notes (none) -> Have: 1
