File: M6/CPR Machine Schematic/Power.kicad_sch (KiCad schematic)
At the start: 52 parts, among them J1 Battery 22.2V IN, J16 Motor Driver, J2 Power Switch, J3 GND Spare Headers, J4 +V Spare Headers, Q1 DMMT5401 PNP, Q2 SSM3J332R, Q3 DMG2305UX-EV, Q4 DMMT5401 PNP, SW1 SW_SPST, U1 3.3V Buck, U2 12V Buck, U3 MAX42403AFLB+

Commit message: Missing cap values
Parts:
- F3: value 40A -> 20A
