File: M6/CPR Machine Schematic/CPR Machine Schematic.kicad_pcb (KiCad board)
At the start: 2 copper layers, 89.9 x 63 mm, 85 parts, among them J1 Battery 22.2V IN, J10 Stop Button Port, J11 Go Button Port, J12 Force Sensor, J13 Laser Port, J14 Raspberry_Pi_2_3, J2 Power Switch, J3 5V Spare Headers, J4 GND Spare Headers, J5 3V3 Spare Headers, J6 12 Spare headers, J7 Battery Spare headers, J8 Conn_02x20_Odd_Even, J9 I2C Port, Q1 DMMT5401 PNP, Q2 SSM3J332R, Q3 DMG2305UX-EV, Q4 DMMT5401 PNP, Q5 T2N7002BK,LM, Q6 T2N7002BK,LM, Q7 T2N7002BK,LM, U1 3.3V Buck, U2 12V Buck, U3 MAX42403AFLB+, U4 MCP6004, U5 MCP3021A0T-E_OT

Commit message: Condensed Header Pins
Parts:
- removed the J5 at (149.3, 77.8)
- removed the J6 at (158.0, 77.8)
- removed the J7 at (164.1, 77.8)
- added C6: 10 nF, Capacitor_SMD:C_1206_3216Metric_Pad1.33x1.80mm_HandSolder, F.Cu at (163.5, 105.0)
- added G***: LOGO, Images:Occam, F.Cu at (165.3, 85.0)
- J3: value 5V Spare Headers -> +V Spare Headers; footprint Connector_PinHeader_2.54mm:PinHeader_1x05_P2.54mm_Vertical -> Connector_PinHeader_2.54mm:PinHeader_1x12_P2.54mm_Vertical
- moved REF** 33.1 mm to (135.6, 98.1)
- moved U1 7.81 mm to (126.8, 100.8)
- moved Q4 2.80 mm to (162.7, 96.4)
- moved Q3 2.77 mm to (163.5, 101.8)
- moved R11 2.40 mm to (158.2, 97.0)
- moved R10 2.25 mm to (158.2, 94.7)
- moved F1 2.00 mm to (128.5, 110.8)
- moved Q1 2.00 mm to (128.7, 116.0)
- moved Q2 2.00 mm to (133.8, 110.5)
- moved R1 2.00 mm to (133.3, 114.9)
- moved R2 2.00 mm to (132.7, 118.5)
- moved REF** 0.55 mm to (158.8, 88.3)
- renumbered C9 to C10, C10 to C11, C6 to C7, C7 to C8, C8 to C9, J13 to J10, J14 to J11, J8 to J5, J9 to J6, J10 to J7, J11 to J8, J12 to J9, R2 to R1, R15 to R14, R14 to R15, R1 to R2, U2 to U1, U1 to U2
Connections:
- C8 pad 2: +3V3 -> +3.3V
- C9 pad 2: +3V3 -> +3.3V
- U4 pad 4: +3V3 -> +3.3V
- U5 pad 1: +3V3 -> +3.3V
Routing:
- net +3.3V: track 186.4 -> 228.5 mm, vias 3 -> 4
- net +3V3: track 13.6 -> 0.00 mm, vias 2 -> 0
- net +12V: track 80.2 -> 72.5 mm
- net GND: track 78.2 -> 85.4 mm
- net /Power/From Switch: track 15.5 -> 8.77 mm
- net +22.2V: track 130.6 -> 125.8 mm
- net Net-(C11-Pad1): track 14.8 -> 11.0 mm
- net /Power/Reg OUT: track 31.6 -> 30.1 mm
- net Net-(J12-Pin_1): track 30.9 -> 32.0 mm, vias 4 -> 2
- net /HMI_Raspi/Laser_PWM: track 91.6 -> 92.4 mm
- net Net-(U5-AIN): track 24.3 -> 24.5 mm, vias 0 -> 2
Other:
- board text added: "Daniel Gliksberg HB Main Board v3"
- board text removed: "Daniel Gliksberg HB Main Board v2"

Commit message: GND testpoint, Main 0V diode redesign, Geograph Redesignate
Parts:
- added TP5: GND, TestPoint:TestPoint_THTPad_4.0x4.0mm_Drill2.0mm, F.Cu at (134.6, 75.7)
- J1, J2: footprint Connector_AMASS:AMASS_XT30PW-M_1x02_P2.50mm_Horizontal -> Connector_AMASS:AMASS_XT30PW-F_1x02_P2.50mm_Horizontal
- TP4: footprint TestPoint:TestPoint_THTPad_4.0x4.0mm_Drill2.0mm -> TestPoint:TestPoint_THTPad_D4.0mm_Drill2.0mm
- moved U2 6.23 mm to (123.4, 95.5), turned to -90 degrees
- moved J2 5.11 mm to (118.5, 102.1)
- moved J1 5.09 mm to (118.5, 116.6)
- moved R1 5.02 mm to (127.8, 117.3), turned to 90 degrees
- moved J3 3.56 mm to (139.2, 74.2)
- moved J4 3.56 mm to (139.2, 77.8)
- moved Q1 2.80 mm to (130.9, 117.6)
- moved R2 2.57 mm to (134.1, 117.3)
- moved TP4 1.23 mm to (129.5, 75.7)
- moved Q2 1.20 mm to (133.1, 111.5)
- moved F1 1.00 mm to (127.9, 111.5)
- moved TP3 0.57 mm to (124.5, 75.7)
- moved TP2 0.06 mm to (118.1, 83.1)
- renumbered C6 to C5, C5 to C6, C9 to C8, C8 to C9, G*** to G***1, G*** to G***2, G*** to G***3, J4 to J3, J3 to J4, LED2 to LED1, LED1 to LED2, Q7 to Q5, Q5 to Q6, Q6 to Q7, R2 to R1, R18 to R14, R14 to R15, R15 to R16, R16 to R17, R17 to R18, R1 to R2, R9 to R6, R8 to R7, R6 to R8, R7 to R9, REF** to REF**1, REF** to REF**2, TP5 to TP6, TP6 to TP7, TP7 to TP8, U2 to U1, U1 to U2
Connections:
- J1 pad 1: /Power/Battery + -> GND
- J1 pad 2: GND -> /Power/Battery +
Routing:
- net +3.3V: track 228.5 -> 244.8 mm, vias 4 -> 6
- net +12V: track 72.5 -> 78.7 mm
- net +22.2V: track 125.8 -> 129.4 mm
- net /Power/From Switch: track 8.77 -> 5.35 mm
- net /HMI_Raspi/Stop_Enable: track 92.7 -> 93.8 mm
- net /HMI_Raspi/Laser_PWM: track 92.4 -> 93.5 mm
- net /HMI_Raspi/Stop Button: track 65.3 -> 66.4 mm
- net /HMI_Raspi/Go_Enable: track 70.5 -> 71.7 mm
- net /HMI_Raspi/Go Button: track 68.3 -> 69.4 mm
- net /Power/Battery +: track 8.84 -> 7.91 mm
- net Net-(Q1-Pad4): track 7.05 -> 7.63 mm
Other:
- board size 89.9 x 63 mm -> 84.1 x 63 mm
