File: M6/CPR Machine Schematic/HMI_Raspi.kicad_sch (KiCad schematic)
At the start: 17 parts, among them J10 Stop Button Port, J11 Go Button Port, J13 Laser Port, Q5 T2N7002BK,LM, Q6 T2N7002BK,LM, Q7 T2N7002BK,LM

Commit message: Condensed Header Pins
Parts:
- renumbered C9 to C10, C10 to C11, J13 to J10, J10 to J7, J11 to J8, R15 to R14, R14 to R15
Changed lines of the file:
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@@
 		(on_board yes)
 		(dnp no)
-		(property "Reference" "J10"
+		(property "Reference" "J7"
 			(at 154.432 39.37 0)
 			(effects
@@
 			(project ""
 				(path "/8991fc77-975f-4978-a089-6b2a5e33f59b/4742a649-a015-487c-b382-01878b0e2dd4"
-					(reference "J10")
+					(reference "J7")
 					(unit 1)
 				)
@@
 		(dnp no)
 		(fields_autoplaced yes)
-		(property "Reference" "J13"
+		(property "Reference" "J10"
 			(at 107.95 53.3399 0)
 			(effects
@@
 			(project ""
 				(path "/8991fc77-975f-4978-a089-6b2a5e33f59b/4742a649-a015-487c-b382-01878b0e2dd4"
-					(reference "J13")
+					(reference "J10")
 					(unit 1)
 				)
@@
 		(on_board yes)
 		(dnp no)
-		(property "Reference" "R14"
+		(property "Reference" "R15"
 			(at 134.62 62.23 90)
 			(effects
@@
 			(project "CPR Machine Schematic"
 				(path "/8991fc77-975f-4978-a089-6b2a5e33f59b/4742a649-a015-487c-b382-01878b0e2dd4"
-					(reference "R14")
+					(reference "R15")
 					(unit 1)
 				)
@@
 		(on_board yes)
 		(dnp no)
-		(property "Reference" "C9"
+		(property "Reference" "C10"
 			(at 135.382 52.07 0)
 			(effects
@@
 			(project ""
 				(path "/8991fc77-975f-4978-a089-6b2a5e33f59b/4742a649-a015-487c-b382-01878b0e2dd4"
-					(reference "C9")
+					(reference "C10")
 					(unit 1)
 				)
@@
 		(on_board yes)
 		(dnp no)
-		(property "Reference" "C10"
+		(property "Reference" "C11"
 			(at 135.382 95.25 0)
 			(effects
@@
 			(project "CPR Machine Schematic"
 				(path "/8991fc77-975f-4978-a089-6b2a5e33f59b/4742a649-a015-487c-b382-01878b0e2dd4"
-					(reference "C10")
+					(reference "C11")
 					(unit 1)
 				)
@@
 		(on_board yes)
 		(dnp no)
-		(property "Reference" "R15"
+		(property "Reference" "R14"
 			(at 132.588 69.088 0)
 			(effects
@@
 			(project "CPR Machine Schematic"
 				(path "/8991fc77-975f-4978-a089-6b2a5e33f59b/4742a649-a015-487c-b382-01878b0e2dd4"
-					(reference "R15")
+					(reference "R14")
 					(unit 1)
 				)
@@
 		(on_board yes)
 		(dnp no)
-		(property "Reference" "J11"
+		(property "Reference" "J8"
 			(at 154.432 78.74 0)
 			(effects
@@
 			(project "CPR Machine Schematic"
 				(path "/8991fc77-975f-4978-a089-6b2a5e33f59b/4742a649-a015-487c-b382-01878b0e2dd4"
-					(reference "J11")
-					(unit 1)
-				)
+					(reference "J8")
+					(unit 1)
+				)

Commit message: Part Inventory
Parts:
- J10: Notes (none) -> Have: 5; now in the parts list
- Q5, Q6, Q7: Notes (none) -> Have: 6
- R19, R20: Notes (none) -> Have: 1; now in the parts list

Commit message: GND testpoint, Main 0V diode redesign, Geograph Redesignate
Parts:
- renumbered Q7 to Q5, Q5 to Q6, Q6 to Q7, R14 to R15, R15 to R16, R16 to R17, R17 to R18
Changed lines of the file:
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@@
 		(on_board yes)
 		(dnp no)
-		(property "Reference" "R15"
+		(property "Reference" "R16"
 			(at 134.62 62.23 90)
 			(effects
@@
 			(project "CPR Machine Schematic"
 				(path "/8991fc77-975f-4978-a089-6b2a5e33f59b/4742a649-a015-487c-b382-01878b0e2dd4"
-					(reference "R15")
+					(reference "R16")
 					(unit 1)
 				)
@@
 		(dnp no)
 		(fields_autoplaced yes)
-		(property "Reference" "Q6"
+		(property "Reference" "Q7"
 			(at 149.86 109.2199 0)
 			(effects
@@
 			(project "CPR Machine Schematic"
 				(path "/8991fc77-975f-4978-a089-6b2a5e33f59b/4742a649-a015-487c-b382-01878b0e2dd4"
-					(reference "Q6")
+					(reference "Q7")
 					(unit 1)
 				)
@@
 		(on_board yes)
 		(dnp no)
-		(property "Reference" "R16"
+		(property "Reference" "R17"
 			(at 134.62 106.68 90)
 			(effects
@@
 			(project "CPR Machine Schematic"
 				(path "/8991fc77-975f-4978-a089-6b2a5e33f59b/4742a649-a015-487c-b382-01878b0e2dd4"
-					(reference "R16")
+					(reference "R17")
 					(unit 1)
 				)
@@
 		(on_board yes)
 		(dnp no)
-		(property "Reference" "R14"
+		(property "Reference" "R15"
 			(at 132.588 69.088 0)
 			(effects
@@
 			(project "CPR Machine Schematic"
 				(path "/8991fc77-975f-4978-a089-6b2a5e33f59b/4742a649-a015-487c-b382-01878b0e2dd4"
-					(reference "R14")
+					(reference "R15")
 					(unit 1)
 				)
@@
 		(dnp no)
 		(fields_autoplaced yes)
-		(property "Reference" "Q7"
+		(property "Reference" "Q5"
 			(at 101.6 62.2299 0)
 			(effects
@@
 			(project "CPR Machine Schematic"
 				(path "/8991fc77-975f-4978-a089-6b2a5e33f59b/4742a649-a015-487c-b382-01878b0e2dd4"
-					(reference "Q7")
+					(reference "Q5")
 					(unit 1)
 				)
@@
 		(dnp no)
 		(fields_autoplaced yes)
-		(property "Reference" "Q5"
+		(property "Reference" "Q6"
 			(at 149.86 64.7699 0)
 			(effects
@@
 			(project "CPR Machine Schematic"
 				(path "/8991fc77-975f-4978-a089-6b2a5e33f59b/4742a649-a015-487c-b382-01878b0e2dd4"
-					(reference "Q5")
+					(reference "Q6")
 					(unit 1)
 				)
@@
 		(on_board yes)
 		(dnp no)
-		(property "Reference" "R17"
+		(property "Reference" "R18"
 			(at 131.318 113.538 0)
 			(effects
@@
 			(project "CPR Machine Schematic"
 				(path "/8991fc77-975f-4978-a089-6b2a5e33f59b/4742a649-a015-487c-b382-01878b0e2dd4"
-					(reference "R17")
+					(reference "R18")
 					(unit 1)
 				)
