File: M6/Contactor Board Schematic/Contactor Board Schematic.kicad_sch (KiCad schematic)
At the start: 12 parts

Commit message: CT board progress
Parts:
- removed J_EXT4: Switch/Contactor, Connector_AMASS:AMASS_XT30PW-F_1x02_P2.50mm_Horizontal, symbol Connector:Conn_01x02_Socket
- added D6: SMCJ15A, Diode_SMD:D_SMC, symbol Device:D_Zener
- added D7: SMCJ28A, Diode_SMD:D_SMC, symbol Device:D_Zener
- added U2: 12V Buck, Converter_DCDC:Converter_DCDC_TRACO_TSR-1_THT, symbol Regulator_Switching:TSR_1-24120
- J_EXT1: footprint Connector_AMASS:AMASS_XT30PW-F_1x02_P2.50mm_Horizontal -> TerminalBlock:TerminalBlock_MaiXu_MX126-5.0-02P_1x02_P5.00mm; digikey (none) -> 277-1667-ND; gobilda 3803-0033-0002 -> (none)
- J_EXT2, J_EXT3, J_EXT5: footprint Connector_AMASS:AMASS_XT30PW-F_1x02_P2.50mm_Horizontal -> Connector_AMASS:AMASS_XT30U-M_1x02_P5.0mm_Vertical
Connections:
- net GND: now also D6.2 (A), D7.2 (A), U2.2 (GND)
- net From Switch renamed Switch
- net Switch: now also D7.1 (K), U2.1 (Vin)
- net To Contactor renamed Contactor
- net Contactor: now also D6.1 (K), U2.3 (Vout)
Other:
- note added: "Screw terminal to EC5 Connector"
- note removed: "Power Cable"
- moved on the sheet: Contactor1, F3, Flyback1, H1, H2, H3, H4

Commit message: Contactor Progress
Parts:
- removed D6: SMCJ15A, Diode_SMD:D_SMC, symbol Device:D_Zener
- removed D7: SMCJ28A, Diode_SMD:D_SMC, symbol Device:D_Zener
- added D2, D4: SMCJ28A, Diode_SMD:D_SMC, symbol Device:D_Zener
- added D6: SMCJ28CA, Diode_SMD:D_SMC, symbol Device:D_TVS
- H1, H2, H3, H4: footprint (none) -> MountingHole:MountingHole_2.7mm_Pad
- renumbered F3 to F1, J_EXT5 to J_EXT2, J_EXT2 to J_EXT3, J_EXT3 to J_EXT4, U2 to U1
Connections:
- net Battery +: now also D6.2 (A2)
- net GND: now also D2.2 (A), D4.2 (A), D6.1 (A1)
- net Switch: now also D4.1 (K)
- net at Contactor1.1, J_EXT1.2 (Pin_2), J_EXT2.1 (Pin_1): now also D2.1 (K)
Other:
- moved on the sheet: U1

Commit message: XT60 connector for battery
Parts:
- J_EXT1: footprint TerminalBlock:TerminalBlock_MaiXu_MX126-5.0-02P_1x02_P5.00mm -> Connector_AMASS:AMASS_XT60-M_1x02_P7.20mm_Vertical
Changed lines of the file:
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@@
 			)
 		)
-		(property "Footprint" "TerminalBlock:TerminalBlock_MaiXu_MX126-5.0-02P_1x02_P5.00mm"
+		(property "Footprint" "Connector_AMASS:AMASS_XT60-M_1x02_P7.20mm_Vertical"
 			(at 16.51 31.75 0)
 			(hide yes)
