File: hardware/pcb/main-board/HMI_Raspi.kicad_sch (KiCad schematic)
At the start: 17 parts, among them J10 Laser Port, J7 Stop Button Port, J8 Go Button Port, Q5 T2N7002BK,LM, Q6 T2N7002BK,LM, Q7 T2N7002BK,LM

Commit message: RS485 Comms
Parts:
- added C30: 100 nF, Capacitor_SMD:C_1206_3216Metric_Pad1.33x1.80mm_HandSolder, symbol Device:C
- added J15: RS485 Port, Connector_JST:JST_PH_S4B-PH-K_1x04_P2.00mm_Horizontal, symbol Connector:Conn_01x04_Socket
- added R34, R35, R36, R38, R39: 10 kOhm, Resistor_SMD:R_1206_3216Metric_Pad1.30x1.75mm_HandSolder, symbol Device:R_US
- added R37: 120 Ohm, Resistor_SMD:R_1206_3216Metric_Pad1.30x1.75mm_HandSolder, symbol Device:R_US
- added U8: THVD1439DR, D8_TEX, symbol THVD1429DT:THVD1429DT
Connections:
- net +3.3V: now also C30.2, R34.2, R35.2, U8.8 (VCC)
- net GND: now also C30.1, J15.4 (Pin_4), R36.1, R38.1, R39.2, U8.5 (GND)
- new net: J15.1 (Pin_1), R37.2, R39.1, U8.7 (B)
- new net: J15.2 (Pin_2), R37.1, R38.2, U8.6 (A)
- new net Screen_Data_Dir: R34.1, R36.2, U8.2 (*RE), U8.3 (DE)
- new net USART_RX: R35.1, U8.1 (R)
- new net USART_TX: U8.4 (D)
- no-connect marks 0 -> 1
Other:
- note added: "Bias Resistors - Populate if motor noise interferes with comms"
- note added: "RS485 Screen Comms"
- note removed: "NOTE: This setup causes buttons to only enable when LED is on"
- moved on the sheet: C10, C11, J10, J7, J8, Q5, Q6, Q7, R15, R16, R17, R18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
