File: hardware/pcb/main-board/Raspi.kicad_sch (KiCad schematic)
At the start: 3 parts, among them J11 Raspberry_Pi_2_3, J5 Conn_02x20_Odd_Even

Commit message: Stepper drivers (real)
Parts:
- F2: value 3A -> 2.6A
Changed lines of the file:
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@@
 			)
 		)
-		(property "Value" "3A"
+		(property "Value" "2.6A"
 			(at 138.43 73.6599 0)
 			(show_name no)

Commit message: Start of CAN-FD
Connections:
- net GPIO10: no longer J11.19 (MOSI0/GPIO10)
- net GPIO11: no longer J11.23 (SCLK0/GPIO11)
- net GPIO8: no longer J11.24 (~{CE0}/GPIO8)
- net GPIO9: no longer J11.21 (MISO0/GPIO9)
- net GPIO14: no longer names the net of J5.8 (Pin_8)
- net GPIO14: no longer J11.8 (GPIO14/TXD)
- net GPIO15: no longer names the net of J5.10 (Pin_10)
- net GPIO15: no longer J11.10 (GPIO15/RXD)
- net GPIO16: no longer names the net of J5.36 (Pin_36)
- net GPIO16: no longer J11.36 (GPIO16)
- net GPIO17: no longer names the net of J5.11 (Pin_11)
- net GPIO17: no longer J11.11 (GPIO17)
- new net CS: J11.24 (~{CE0}/GPIO8)
- new net Dir: J11.36 (GPIO16)
- new net MISO: J11.21 (MISO0/GPIO9)
- new net MOSI: J11.19 (MOSI0/GPIO10)
- new net SCK: J11.23 (SCLK0/GPIO11)
- new net Step: J11.11 (GPIO17)
- new net Stepper Enable: J11.8 (GPIO14/TXD)
- new net Stepper Sleep: J11.10 (GPIO15/RXD)
- no-connect marks 9 -> 13
Changed lines of the file:
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@@
+	)
+	(no_connect
+		(at 210.82 93.98)
 	)
 	(no_connect
@@
 	)
 	(no_connect
+		(at 210.82 96.52)
+	)
+	(no_connect
 		(at 198.12 91.44)
 	)
@@
 	)
 	(no_connect
+		(at 210.82 129.54)
+	)
+	(no_connect
 		(at 210.82 111.76)
 	)
@@
 	)
 	(no_connect
+		(at 198.12 99.06)
+	)
+	(no_connect
 		(at 143.51 77.47)
 	)
@@
 			(width 0)
 			(type default)
-		)
-	)
-	(label "GPIO16"
-		(at 210.82 129.54 0)
-		(effects
-			(font
-				(size 1.27 1.27)
-			)
-			(justify left bottom)
 		)
 	)
@@
 		)
 	)
-	(label "GPIO17"
-		(at 198.12 99.06 180)
-		(effects
-			(font
-				(size 1.27 1.27)
-			)
-			(justify right bottom)
-		)
-	)
 	(label "GPIO13"
 		(at 161.29 130.81 0)
@@
 		)
 	)
-	(label "GPIO16"
-		(at 120.65 95.25 180)
-		(effects
-			(font
-				(size 1.27 1.27)
-			)
-			(justify right bottom)
-		)
-	)
 	(label "GPIO20"
 		(at 210.82 132.08 0)
@@
 		)
 	)
-	(label "GPIO10"
-		(at 161.29 120.65 0)
-		(effects
-			(font
-				(size 1.27 1.27)
-			)
-			(justify left bottom)
-		)
-	)
 	(label "GPIO0"
 		(at 198.12 119.38 180)
@@
 		)
 	)
-	(label "GPIO9"
-		(at 161.29 118.11 0)
-		(effects
-			(font
-				(size 1.27 1.27)
-			)
-			(justify left bottom)
-		)
-	)
 	(label "GPIO0"
 		(at 161.29 87.63 0)
@@
 		)
 	)
-	(label "GPIO17"
-		(at 120.65 97.79 180)
-		(effects
-			(font
-				(size 1.27 1.27)
-			)
-			(justify right bottom)
-		)
-	)
 	(label "GPIO7"
 		(at 161.29 113.03 0)
@@
 		)
 	)
-	(label "GPIO15"
-		(at 210.82 96.52 0)
-		(effects
-			(font
-				(size 1.27 1.27)
-			)
-			(justify left bottom)
-		)
-	)
-	(label "GPIO15"
-		(at 120.65 90.17 180)
-		(effects
-			(font
-				(size 1.27 1.27)
-			)
-			(justify right bottom)
-		)
-	)
-	(label "GPIO14"
-		(at 210.82 93.98 0)
-		(effects
-			(font
-				(size 1.27 1.27)
-			)
-			(justify left bottom)
-		)
-	)
 	(label "GPIO8"
 		(at 210.82 114.3 0)
@@
 		)
 	)
-	(label "GPIO14"
-		(at 120.65 87.63 180)
-		(effects
-			(font
-				(size 1.27 1.27)
-			)
-			(justify right bottom)
-		)
-	)
 	(label "GPIO20"
 		(at 120.65 107.95 180)
@@
 		)
 	)
-	(label "GPIO11"
-		(at 161.29 123.19 0)
-		(effects
-			(font
-				(size 1.27 1.27)
-			)
-			(justify left bottom)
-		)
-	)
 	(label "GPIO22"
 		(at 198.12 104.14 180)
@@
 		)
 	)
-	(label "GPIO8"
-		(at 161.29 115.57 0)
-		(effects
-			(font
-				(size 1.27 1.27)
-			)
-			(justify left bottom)
-		)
-	)
 	(label "GPIO13"
 		(at 198.12 127 180)
@@
 			)
 			(justify right bottom)
+		)
+	)
+	(hierarchical_label "Stepper Enable"
+		(shape output)
+		(at 120.65 87.63 180)
+		(effects
+			(font
+				(size 1.27 1.27)
+			)
+			(justify right)
+		)
+	)
+	(hierarchical_label "SCK"
+		(shape output)
+		(at 161.29 123.19 0)
+		(effects
+			(font
+				(size 1.27 1.27)
+			)
+			(justify left)
 		)
 	)
@@
 		)
 	)
+	(hierarchical_label "Stepper Sleep"
+		(shape output)
+		(at 120.65 90.17 180)
+		(effects
+			(font
+				(size 1.27 1.27)
+			)
+			(justify right)
+		)
+	)
 	(hierarchical_label "Go_Button"
 		(shape output)
@@
 			)
 			(justify right)
+		)
+	)
+	(hierarchical_label "CS"
+		(shape output)
+		(at 161.29 115.57 0)
+		(effects
+			(font
+				(size 1.27 1.27)
+			)
+			(justify left)
 		)
 	)
@@
 		)
 	)
+	(hierarchical_label "Dir"
+		(shape output)
+		(at 120.65 95.25 180)
+		(effects
+			(font
+				(size 1.27 1.27)
+			)
+			(justify right)
+		)
+	)
 	(hierarchical_label "Stop_Button"
 		(shape output)
@@
 		)
 	)
+	(hierarchical_label "MISO"
+		(shape input)
+		(at 161.29 118.11 0)
+		(effects
+			(font
+				(size 1.27 1.27)
+			)
+			(justify left)
+		)
+	)
 	(hierarchical_label "Stop_Enable"
 		(shape output)
@@
 		(effects
 			(font
+				(size 1.27 1.27)
+			)
+			(justify right)
+		)
+	)
+	(hierarchical_label "MOSI"
+		(shape output)
+		(at 161.29 120.65 0)
+		(effects
+			(font
+				(size 1.27 1.27)
+			)
+			(justify left)
+		)
+	)
+	(hierarchical_label "Step"
+		(shape output)
+		(at 120.65 97.79 180)
+		(effects
+			(font

Commit message: CAN-FD Transceiver Done
Connections:
- net CS: no longer names the net of J11.24 (~{CE0}/GPIO8)
- net MISO renamed RX_CAN
- net MOSI renamed TX_CAN
- net SCK renamed CAN Standby
Other:
- note removed: "Screens and Motor Driver connected via HDMI and USB Ports, not GPIO"
Changed lines of the file:
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@@
 	(generator_version "10.0")
 	(paper "A4")
-	(rectangle
-		(start 13.335 13.335)
-		(end 83.82 15.875)
-		(stroke
-			(width 0)
-			(type default)
-		)
-		(fill
-			(type none)
-		)
-	)
 	(text "Spare GPIO\nHeader"
 		(exclude_from_sim no)
@@
 		)
 	)
-	(text "Screens and Motor Driver connected via HDMI and USB Ports, not GPIO"
-		(exclude_from_sim no)
-		(at 48.514 14.986 0)
-		(effects
-			(font
-				(size 1.27 1.27)
-			)
-		)
-	)
 	(text "3V3 disconnected because of seperate 3V3 source on hat"
 		(exclude_from_sim no)
@@
 		)
 	)
-	(hierarchical_label "SCK"
-		(shape output)
-		(at 161.29 123.19 0)
-		(effects
-			(font
-				(size 1.27 1.27)
-			)
-			(justify left)
-		)
-	)
 	(hierarchical_label "I2C_SDA"
 		(shape bidirectional)
@@
 		)
 	)
-	(hierarchical_label "CS"
-		(shape output)
-		(at 161.29 115.57 0)
+	(hierarchical_label "TX_CAN"
+		(shape input)
+		(at 161.29 120.65 0)
 		(effects
 			(font
@@
 		)
 	)
-	(hierarchical_label "MISO"
+	(hierarchical_label "RX_CAN"
 		(shape input)
 		(at 161.29 118.11 0)
@@
 		)
 	)
-	(hierarchical_label "MOSI"
-		(shape output)
-		(at 161.29 120.65 0)
+	(hierarchical_label "Step"
+		(shape output)
+		(at 120.65 97.79 180)
+		(effects
+			(font
+				(size 1.27 1.27)
+			)
+			(justify right)
+		)
+	)
+	(hierarchical_label "CAN Standby"
+		(shape output)
+		(at 161.29 123.19 0)
 		(effects
 			(font
@@
 		)
 	)
-	(hierarchical_label "Step"
-		(shape output)
-		(at 120.65 97.79 180)
-		(effects
-			(font
-				(size 1.27 1.27)
-			)
-			(justify right)
-		)
-	)

Commit message: IMUs, I2C Pullups, Screen Power USB-C Ports
Parts:
- added R44, R45: 10k, Resistor_SMD:R_1206_3216Metric_Pad1.30x1.75mm_HandSolder, symbol Device:R_US
- F2: value 2.6A -> 3A
Connections:
- net +3.3V: now also R44.2, R45.1
- net I2C_SCL: now also R45.2
- net I2C_SDA: now also R44.1
