File: hardware/pcb/main-board/Sensing.kicad_sch (KiCad schematic)
At the start: 20 parts, among them J6 I2C Port, J9 Force Sensor, U4 MCP6004, U5 MCP3021A5T-E_OT

Commit message: IMUs, I2C Pullups, Screen Power USB-C Ports
Parts:
- added C31, C32, C33, C34: 0.1 uF, Capacitor_SMD:C_1206_3216Metric_Pad1.33x1.80mm_HandSolder, symbol Device:C
- added U10, U2: LSM6DSV16XTR, Package_LGA:LGA-14_3x2.5mm_P0.5mm_LayoutBorder3x4y, symbol 2026-10-29_17-21-07:LSM6DSV16XTR
Connections:
- net +3.3V: now also C31.2, C32.2, C33.2, C34.2, U10.1 (SDO/SA0), U10.12 (CS), U10.5 (VDD_IO), U10.8 (VDD), U2.12 (CS), U2.5 (VDD_IO), U2.8 (VDD)
- net GND: now also C31.1, C32.1, C33.1, C34.1, U10.2 (SDX/AH1/QVAR1), U10.3 (SCX/AH2/QVAR2), U10.6 (GND), U10.7 (GND), U2.1 (SDO/SA0), U2.2 (SDX/AH1/QVAR1), U2.3 (SCX/AH2/QVAR2), U2.6 (GND), U2.7 (GND)
- net I2C_SCL: now also U10.13 (SCL), U2.13 (SCL)
- net I2C_SDA: now also U10.14 (SDA), U2.14 (SDA)
- no-connect marks 0 -> 8
Other:
- note added: "IMUs"
